File: SwedishChainsaw.kicad_pcb (KiCad board)
At the start: 2 copper layers, 59 x 60.5 mm, 77 parts, among them Q1 NJFET, Q2 2N3904, Q3 2N3906, U1 TL072, U2 TL072, U3 TL072

Commit message: Add files via upload
Other:
- board text added: "CHAINSAW"

Commit message: Add files via upload
Parts:
- added G***: LOGO, LOGO, F.Cu at (49.4, 60.4)
- added G***: LOGO, LOGO, B.Cu at (51.4, 60.4)
- moved OUT 7.15 mm to (67.7, 113.0)
Connections:
- RV1 pad : (no net) -> GND
- RV2 pad : (no net) -> GND
- RV3 pad : (no net) -> GND
- RV4 pad : (no net) -> GND
Routing:
- net /out: track 19.6 -> 27.4 mm
- net /Vin: track 8.88 -> 10.1 mm
- net Net-(U3B-+): track 111.7 -> 112.9 mm
Other:
- board text added: "JLCJLCJLCJLC"
- board text added: "KJ"
